File: board/servo_driver.kicad_sch (KiCad schematic)
At the start: 27 parts, among them U5 PCA9685PW

Commit message: More work on PCB design
Parts:
- removed JP1, JP2, JP3, JP4: SolderJumper_2_Open, Jumper:SolderJumper-2_P1.3mm_Open_Pad1.0x1.5mm, symbol Jumper:SolderJumper_2_Open
Connections:
- net +5V: now also conn_3x4.11, conn_3x4.2, conn_3x4.5, conn_3x4.8
Changed lines of the file:
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@@
     (fill (type none))
-  )
-  (text_box "Last 4 servos shouldn't be connected to VCC. They are ought to be used to controll BLCD motors ESC with high noisy 5V"
-    (at 210.82 144.78 0) (size 46.355 10.16)
-    (stroke (width 0) (type default))
-    (fill (type none))
-    (effects (font (size 1.27 1.27) bold) (justify left top))
   )
   (text "PCA9685" (at 27.305 55.245 0)
@@
     )
   )
-  (symbol (lib_id "Jumper:SolderJumper_2_Open") (at 237.49 127 0) (unit 1)
-    (in_bom yes) (on_board yes) (dnp no)
-    (property "Reference" "JP3" (at 238.76 123.19 0)
-      (effects (font (size 1.27 1.27)))
-    )
-    (property "Value" "SolderJumper_2_Open" (at 243.205 125.095 0)
-      (effects (font (size 1.27 1.27)))
-    )
-    (property "Footprint" "Jumper:SolderJumper-2_P1.3mm_Open_Pad1.0x1.5mm" (at 237.49 127 0)
-      (effects (font (size 1.27 1.27)) hide)
-    )
-    (property "Datasheet" "~" (at 237.49 127 0)
-      (effects (font (size 1.27 1.27)) hide)
-    )
-    (pin "1")
-    (pin "2")
-    (instances
-      (project "uav_project"
-        (path "/a8bf0924-b264-4c19-8c7e-9c0e131cacba/46d9e855-1ab1-4192-9cab-93e4258e1e2b"
-          (reference "JP3") (unit 1)
-        )
-      )
-    )
-  )
   (symbol (lib_id "power:+5V") (at 233.68 93.98 270) (unit 1)
     (in_bom yes) (on_board yes) (dnp no) (fields_autoplaced)
@@
     )
   )
-  (symbol (lib_id "power:+5V") (at 241.3 109.22 270) (unit 1)
-    (in_bom yes) (on_board yes) (dnp no) (fields_autoplaced)
-    (property "Reference" "#PWR074" (at 237.49 109.22 0)
-      (effects (font (size 1.27 1.27)) hide)
-    )
-    (property "Value" "+5V" (at 245.11 109.22 90)
-      (effects (font (size 1.27 1.27)) (justify left))
-    )
-    (property "Footprint" "" (at 241.3 109.22 0)
-      (effects (font (size 1.27 1.27)) hide)
-    )
-    (property "Datasheet" "" (at 241.3 109.22 0)
+  (symbol (lib_id "power:+5V") (at 233.68 109.22 270) (unit 1)
+    (in_bom yes) (on_board yes) (dnp no) (fields_autoplaced)
+    (property "Reference" "#PWR074" (at 229.87 109.22 0)
+      (effects (font (size 1.27 1.27)) hide)
+    )
+    (property "Value" "+5V" (at 237.49 109.22 90)
+      (effects (font (size 1.27 1.27)) (justify left))
+    )
+    (property "Footprint" "" (at 233.68 109.22 0)
+      (effects (font (size 1.27 1.27)) hide)
+    )
+    (property "Datasheet" "" (at 233.68 109.22 0)
       (effects (font (size 1.27 1.27)) hide)
     )
@@
     )
   )
-  (symbol (lib_id "power:+5V") (at 241.3 118.11 270) (unit 1)
-    (in_bom yes) (on_board yes) (dnp no) (fields_autoplaced)
-    (property "Reference" "#PWR076" (at 237.49 118.11 0)
-      (effects (font (size 1.27 1.27)) hide)
-    )
-    (property "Value" "+5V" (at 245.11 118.11 90)
-      (effects (font (size 1.27 1.27)) (justify left))
-    )
-    (property "Footprint" "" (at 241.3 118.11 0)
-      (effects (font (size 1.27 1.27)) hide)
-    )
-    (property "Datasheet" "" (at 241.3 118.11 0)
+  (symbol (lib_id "power:+5V") (at 233.68 118.11 270) (unit 1)
+    (in_bom yes) (on_board yes) (dnp no) (fields_autoplaced)
+    (property "Reference" "#PWR076" (at 229.87 118.11 0)
+      (effects (font (size 1.27 1.27)) hide)
+    )
+    (property "Value" "+5V" (at 237.49 118.11 90)
+      (effects (font (size 1.27 1.27)) (justify left))
+    )
+    (property "Footprint" "" (at 233.68 118.11 0)
+      (effects (font (size 1.27 1.27)) hide)
+    )
+    (property "Datasheet" "" (at 233.68 118.11 0)
       (effects (font (size 1.27 1.27)) hide)
     )
@@
         (path "/a8bf0924-b264-4c19-8c7e-9c0e131cacba/46d9e855-1ab1-4192-9cab-93e4258e1e2b"
           (reference "R13") (unit 1)
-        )
-      )
-    )
-  )
-  (symbol (lib_id "Jumper:SolderJumper_2_Open") (at 237.49 118.11 0) (unit 1)
-    (in_bom yes) (on_board yes) (dnp no)
-    (property "Reference" "JP2" (at 238.76 114.3 0)
-      (effects (font (size 1.27 1.27)))
-    )
-    (property "Value" "SolderJumper_2_Open" (at 243.205 116.205 0)
-      (effects (font (size 1.27 1.27)))
-    )
-    (property "Footprint" "Jumper:SolderJumper-2_P1.3mm_Open_Pad1.0x1.5mm" (at 237.49 118.11 0)
-      (effects (font (size 1.27 1.27)) hide)
-    )
-    (property "Datasheet" "~" (at 237.49 118.11 0)
-      (effects (font (size 1.27 1.27)) hide)
-    )
-    (pin "1")
-    (pin "2")
-    (instances
-      (project "uav_project"
-        (path "/a8bf0924-b264-4c19-8c7e-9c0e131cacba/46d9e855-1ab1-4192-9cab-93e4258e1e2b"
-          (reference "JP2") (unit 1)
         )
       )
@@
     )
   )
-  (symbol (lib_id "power:+5V") (at 241.3 127 270) (unit 1)
-    (in_bom yes) (on_board yes) (dnp no) (fields_autoplaced)
-    (property "Reference" "#PWR077" (at 237.49 127 0)
-      (effects (font (size 1.27 1.27)) hide)
-    )
-    (property "Value" "+5V" (at 245.11 127 90)
-      (effects (font (size 1.27 1.27)) (justify left))
-    )
-    (property "Footprint" "" (at 241.3 127 0)
-      (effects (font (size 1.27 1.27)) hide)
-    )
-    (property "Datasheet" "" (at 241.3 127 0)
+  (symbol (lib_id "power:+5V") (at 233.68 127 270) (unit 1)
+    (in_bom yes) (on_board yes) (dnp no) (fields_autoplaced)
+    (property "Reference" "#PWR077" (at 229.87 127 0)
+      (effects (font (size 1.27 1.27)) hide)
+    )
+    (property "Value" "+5V" (at 237.49 127 90)
+      (effects (font (size 1.27 1.27)) (justify left))
+    )
+    (property "Footprint" "" (at 233.68 127 0)
+      (effects (font (size 1.27 1.27)) hide)
+    )
+    (property "Datasheet" "" (at 233.68 127 0)
       (effects (font (size 1.27 1.27)) hide)
     )
@@
     )
   )
-  (symbol (lib_id "power:+5V") (at 241.3 135.89 270) (unit 1)
-    (in_bom yes) (on_board yes) (dnp no) (fields_autoplaced)
-    (property "Reference" "#PWR078" (at 237.49 135.89 0)
-      (effects (font (size 1.27 1.27)) hide)
-    )
-    (property "Value" "+5V" (at 245.11 135.89 90)
-      (effects (font (size 1.27 1.27)) (justify left))
-    )
-    (property "Footprint" "" (at 241.3 135.89 0)
-      (effects (font (size 1.27 1.27)) hide)
-    )
-    (property "Datasheet" "" (at 241.3 135.89 0)
+  (symbol (lib_id "power:+5V") (at 233.68 135.89 270) (unit 1)
+    (in_bom yes) (on_board yes) (dnp no) (fields_autoplaced)
+    (property "Reference" "#PWR078" (at 229.87 135.89 0)
+      (effects (font (size 1.27 1.27)) hide)
+    )
+    (property "Value" "+5V" (at 237.49 135.89 90)
+      (effects (font (size 1.27 1.27)) (justify left))
+    )
+    (property "Footprint" "" (at 233.68 135.89 0)
+      (effects (font (size 1.27 1.27)) hide)
+    )
+    (property "Datasheet" "" (at 233.68 135.89 0)
       (effects (font (size 1.27 1.27)) hide)
     )
@@
         (path "/a8bf0924-b264-4c19-8c7e-9c0e131cacba/46d9e855-1ab1-4192-9cab-93e4258e1e2b"
           (reference "#PWR078") (unit 1)
-        )
-      )
-    )
-  )
-  (symbol (lib_id "Jumper:SolderJumper_2_Open") (at 237.49 135.89 0) (unit 1)
-    (in_bom yes) (on_board yes) (dnp no)
-    (property "Reference" "JP4" (at 238.76 132.08 0)
-      (effects (font (size 1.27 1.27)))
-    )
-    (property "Value" "SolderJumper_2_Open" (at 243.205 133.985 0)
-      (effects (font (size 1.27 1.27)))
-    )
-    (property "Footprint" "Jumper:SolderJumper-2_P1.3mm_Open_Pad1.0x1.5mm" (at 237.49 135.89 0)
-      (effects (font (size 1.27 1.27)) hide)
-    )
-    (property "Datasheet" "~" (at 237.49 135.89 0)
-      (effects (font (size 1.27 1.27)) hide)
-    )
-    (pin "1")
-    (pin "2")
-    (instances
-      (project "uav_project"
-        (path "/a8bf0924-b264-4c19-8c7e-9c0e131cacba/46d9e855-1ab1-4192-9cab-93e4258e1e2b"
-          (reference "JP4") (unit 1)
         )
       )
@@
         )
       )
-    )
-  )
-  (symbol (lib_id "Jumper:SolderJumper_2_Open") (at 237.49 109.22 0) (unit 1)
-    (in_bom yes) (on_board yes) (dnp no)
-    (property "Reference" "JP1" (at 238.76 105.41 0)
-      (effects (font (size 1.27 1.27)))
-    )
-    (property "Value" "SolderJumper_2_Open" (at 243.205 107.315 0)
-      (effects (font (size 1.27 1.27)))
-    )
-    (property "Footprint" "Jumper:SolderJumper-2_P1.3mm_Open_Pad1.0x1.5mm" (at 237.49 109.22 0)
-      (effects (font (size 1.27 1.27)) hide)
-    )
-    (property "Datasheet" "~" (at 237.49 109.22 0)
-      (effects (font (size 1.27 1.27)) hide)
-    )
-    (pin "1")
-    (pin "2")
-    (instances
-      (project "uav_project"
-        (path "/a8bf0924-b264-4c19-8c7e-9c0e131cacba/46d9e855-1ab1-4192-9cab-93e4258e1e2b"
-          (reference "JP1") (unit 1)
-        )
-      )

Commit message: First version of PCB finished
Connections:
- net +5V: now also U5.2 (A1); no longer U5.24 (A5), U5.4 (A3)
- net GND: now also U5.24 (A5), U5.4 (A3); no longer U5.2 (A1)
- net PWM4: now also R14.2; no longer R11.2
- net PWM5: now also R13.2; no longer R12.2
- net PWM6: now also R12.2; no longer R13.2
- net PWM7: now also R11.2; no longer R14.2
- net at R11.1: now also conn_3x3.10; no longer conn_3x3.1
- net at conn_3x2.1: now also R18.1; no longer R15.1
- net at conn_3x2.10: now also R15.1; no longer R18.1
- net at conn_3x2.4: now also R17.1; no longer R16.1
- net at conn_3x2.7: now also R16.1; no longer R17.1
- net at R13.1: now also conn_3x3.4; no longer conn_3x3.7
- net at R21.1: now also conn_3x4.4; no longer conn_3x4.7
- net at conn_3x4.1: now also R22.1; no longer R19.1
- net at conn_3x4.10: now also R19.1; no longer R22.1
- net at R20.1: now also conn_3x4.7; no longer conn_3x4.4
- net at R14.1: now also conn_3x3.1; no longer conn_3x3.10
- net at R12.1: now also conn_3x3.7; no longer conn_3x3.4
Other:
- moved on the sheet: R11, R12, R13, R14, R15, R16, R17, R18, R19, R20, R21, R22

Commit message: Minor improvements to board design
Parts:
- renumbered conn_3x1 to PWM1, conn_3x3 to PWM2, conn_3x2 to PWM3, conn_3x4 to PWM4
Changed lines of the file:
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@@
   (symbol (lib_name "conn_03x04_Pin_1") (lib_id "Custom_Symbols:conn_03x04_Pin") (at 176.53 62.23 0) (unit 1)
     (in_bom yes) (on_board yes) (dnp no) (fields_autoplaced)
-    (property "Reference" "conn_3x1" (at 177.165 59.69 0)
+    (property "Reference" "PWM1" (at 177.165 59.69 0)
       (effects (font (size 1.27 1.27)))
     )
@@
       (project "uav_project"
         (path "/a8bf0924-b264-4c19-8c7e-9c0e131cacba/46d9e855-1ab1-4192-9cab-93e4258e1e2b"
-          (reference "conn_3x1") (unit 1)
+          (reference "PWM1") (unit 1)
         )
       )
@@
   (symbol (lib_name "conn_03x04_Pin_1") (lib_id "Custom_Symbols:conn_03x04_Pin") (at 227.33 62.23 0) (unit 1)
     (in_bom yes) (on_board yes) (dnp no) (fields_autoplaced)
-    (property "Reference" "conn_3x2" (at 227.965 59.69 0)
+    (property "Reference" "PWM3" (at 227.965 59.69 0)
       (effects (font (size 1.27 1.27)))
     )
@@
       (project "uav_project"
         (path "/a8bf0924-b264-4c19-8c7e-9c0e131cacba/46d9e855-1ab1-4192-9cab-93e4258e1e2b"
-          (reference "conn_3x2") (unit 1)
+          (reference "PWM3") (unit 1)
         )
       )
@@
   (symbol (lib_name "conn_03x04_Pin_1") (lib_id "Custom_Symbols:conn_03x04_Pin") (at 227.33 104.14 0) (unit 1)
     (in_bom yes) (on_board yes) (dnp no) (fields_autoplaced)
-    (property "Reference" "conn_3x4" (at 227.965 101.6 0)
+    (property "Reference" "PWM4" (at 227.965 101.6 0)
       (effects (font (size 1.27 1.27)))
     )
@@
       (project "uav_project"
         (path "/a8bf0924-b264-4c19-8c7e-9c0e131cacba/46d9e855-1ab1-4192-9cab-93e4258e1e2b"
-          (reference "conn_3x4") (unit 1)
+          (reference "PWM4") (unit 1)
         )
       )
@@
   (symbol (lib_name "conn_03x04_Pin_1") (lib_id "Custom_Symbols:conn_03x04_Pin") (at 176.53 104.14 0) (unit 1)
     (in_bom yes) (on_board yes) (dnp no) (fields_autoplaced)
-    (property "Reference" "conn_3x3" (at 177.165 101.6 0)
+    (property "Reference" "PWM2" (at 177.165 101.6 0)
       (effects (font (size 1.27 1.27)))
     )
@@
       (project "uav_project"
         (path "/a8bf0924-b264-4c19-8c7e-9c0e131cacba/46d9e855-1ab1-4192-9cab-93e4258e1e2b"
-          (reference "conn_3x3") (unit 1)
-        )
-      )
+          (reference "PWM2") (unit 1)
+        )
+      )
